Commit message: Added camera to berth fixture

File: astrobee/description/media/astroberth/urdf/model.urdf (robot description, URDF)
Before this commit: robot Berth Fixture V4 Shell.SLDASM, 5 links, 4 joints
Links:
- added link camera_link; visual box size=0.010 0.03 0.03
- added link camera_link_optical
Joints:
- added joint camera_joint: type fixed, parent base_link, child camera_link, origin xyz=0.1 -1 0.175 rpy=0 0 0, axis 0 1 0
- added joint camera_optical_joint: type fixed, parent camera_link, child camera_link_optical, origin xyz=0 0 0 rpy=-1.5707963268 0 -1.5707963268

Commit message: Fixed camera and berth links

File: astrobee/description/media/astroberth/urdf/model.urdf (robot description, URDF)
Before this commit: robot Berth Fixture V4 Shell.SLDASM, 7 links, 6 joints
Joints:
- joint camera_joint: origin xyz=0.1 -1 0.175 rpy=0 0 0 -> xyz=0.1 -1 0.175 rpy=-3.14 0 0

Commit message: fixed cam housing

File: astrobee/description/media/astroberth/urdf/model.urdf (robot description, URDF)
Before this commit: robot Berth Fixture V4 Shell.SLDASM, 7 links, 6 joints
Joints:
- joint camera_joint: origin xyz=0.1 -1 0.175 rpy=-3.14 0 0 -> xyz=-1.5 -1 0.5 rpy=3.14 -0.610865 0

Commit message: Change orientation of camera

File: astrobee/description/media/astroberth/urdf/model.urdf (robot description, URDF)
Before this commit: robot Berth Fixture V4 Shell.SLDASM, 7 links, 6 joints
Joints:
- joint camera_joint: origin xyz=-1.5 -1 0.5 rpy=3.14 -0.610865 0 -> xyz=-1.9 -1.1 0.2 rpy=3.14 -0.410865 0
